File: cwc5.5.kicad_pcb (KiCad board)
At the start: 2 copper layers, 69 x 53 mm, 97 parts, among them J1 Conn_01x08, J2 Conn_01x08, J3 Conn_01x08, J4 Conn_01x07, J5 Conn_01x14, J6 Conn_02x07_Odd_Even, Q1 BC847, Q10 BC847, Q11 BC847, Q12 BC847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

Commit message: Projeto enviado
Parts:
- removed G1: LOGO, User_defined:qr_code
Other:
- board text added: "Github: Ruanfc/cwc_circulating_water_channel"
